File: docs/kiCad/bilgeAlarm.kicad_pcb (KiCad board)
At the start: 2 copper layers, 111.8 x 88.9 mm, 55 parts, among them J1 PUMP IN, J10 LCD_SDA, J11 LCD_SCL, J12 LCD_GND, J13 ALARM+, J14 ALARM-, J15 LED_GND, J16 LED_GND, J17 LED_DATA, J18 LED_DATA, J19 LED_5V, J2 PUMP2 IN, J20 LED_5V, J21 AUX, J22 AUX, J23 AUX, J24 AUX, J25 AUX, J26 AUX, J27 AUX, J28 AUX, J3 PUMP OUT, J4 12V, J5 GND, J6 LED_5V, J7 LED_DATA, J8 LED_GND, J9 LCD_5V, K1 RELAY, M1 BUCK01, M2 SD_TYP0, Q1 IRLZ44N, Q2 BCS547, SW1 POWER, SW2 BUTTON1, SW3 BUTTON2, SW4 BUTTON3, SW5 BUTTON4, U1 ESP32_DEV_0

Commit message: generate flatcam gcode files
Routing:
- net SDA: track 107.6 -> 109.7 mm

Commit message: minor final changes before printing bilgeAlarm PCB
Parts:
- removed SW5: BUTTON4, cnc3018-PCB:BUTTON
- added J29: AUX, cnc3018-PCB:my1pin, F.Cu at (66.0, -38.1)
- added J30: AUX, cnc3018-PCB:my1pin, F.Cu at (101.6, -49.5)
- added J31: AUX, cnc3018-PCB:my1pin, F.Cu at (101.6, -47.0)
- added J32: AUX, cnc3018-PCB:my1pin, F.Cu at (101.6, -44.5)
- added J33: AUX, cnc3018-PCB:my1pin, F.Cu at (101.6, -41.9)
- added J34: AUX, cnc3018-PCB:my1pin, F.Cu at (101.6, -39.4)
- added J35: AUX, cnc3018-PCB:my1pin, F.Cu at (101.6, -36.8)
- added J36: AUX, cnc3018-PCB:my1pin, F.Cu at (104.1, -49.5)
- added J37: AUX, cnc3018-PCB:my1pin, F.Cu at (104.1, -47.0)
- added J38: AUX, cnc3018-PCB:my1pin, F.Cu at (104.1, -44.5)
- added J39: AUX, cnc3018-PCB:my1pin, F.Cu at (104.1, -41.9)
- added J40: AUX, cnc3018-PCB:my1pin, F.Cu at (104.1, -39.4)
- added J41: AUX, cnc3018-PCB:my1pin, F.Cu at (104.1, -36.8)
- moved SW4 7.62 mm to (87.6, -48.3)
- moved SW3 5.08 mm to (69.8, -48.3)
- moved J24 2.54 mm to (63.5, -38.1)
- moved SW2 2.54 mm to (52.1, -48.3)
- moved J15 1.27 mm to (20.3, -85.1)
- moved J17 1.27 mm to (22.9, -85.1)
- moved J19 1.27 mm to (25.4, -85.1)
Connections:
- U1 pad 10: BUTTON4 -> BUTTON3
- U1 pad 5: BUTTON2 -> Net-(J24-Pad1)
- U1 pad 6: Net-(J24-Pad1) -> Net-(J29-Pad1)
- U1 pad 9: BUTTON3 -> BUTTON2
Routing:
- net BUTTON4: track 26.5 -> 0.00 mm
- net +3V3: track 158.2 -> 150.4 mm
- net BUTTON3: track 14.6 -> 21.9 mm
- net +5V: track 163.2 -> 168.4 mm, vias 4 -> 6
- net +12V: track 21.4 -> 25.3 mm, vias 0 -> 1
- net SD_CS: track 30.5 -> 33.0 mm, vias 2 -> 3
- net SDA: track 109.7 -> 112.3 mm, vias 2 -> 3
- net SCL: track 108.3 -> 110.8 mm, vias 2 -> 3
- net Net-(J35-Pad1): track 0.00 -> 2.54 mm
- net Net-(J34-Pad1): track 0.00 -> 2.54 mm
- net Net-(J33-Pad1): track 0.00 -> 2.54 mm
- net Net-(J32-Pad1): track 0.00 -> 2.54 mm
- net Net-(J31-Pad1): track 0.00 -> 2.54 mm
- net Net-(J30-Pad1): track 0.00 -> 2.54 mm
- net Net-(J29-Pad1): track 0.00 -> 2.54 mm
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