File: docs/kiCad/led_board/led_board.sch (KiCad schematic (older format))
At the start: 8 parts, among them J1 Conn_01x03, J2 Conn_01x03, J3 Conn_01x01, J4 Conn_01x01

Commit message: bilgeAlarm led_board v2
Parts:
- D1, D2, D3, D4: footprint LED_SMD:LED_WS2812B_PLCC4_5.0x5.0mm_P3.2mm -> cnc3018-PCB:myWS2812
Connections:
- net at D1.1 (VDD), D2.1 (VDD), D3.1 (VDD)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: now also J1.3 (Pin_3), J2.1 (Pin_1); no longer J1.1 (Pin_1), J2.3 (Pin_3)
- net at D1.3 (VSS), D2.3 (VSS), D3.3 (VSS)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: now also J1.1 (Pin_1), J2.3 (Pin_3); no longer J1.3 (Pin_3), J2.1 (Pin_1)
Other:
- moved on the sheet: J1, J3, J4
Changed lines of the file:
@@
 F 0 "D4" V 2796 4306 50  0000 R CNN
 F 1 "WS2812B" V 2705 4306 50  0000 R CNN
-F 2 "LED_SMD:LED_WS2812B_PLCC4_5.0x5.0mm_P3.2mm" H 2800 4350 50  0001 L TNN
+F 2 "cnc3018-PCB:myWS2812" H 2800 4350 50  0001 L TNN
 F 3 "https://cdn-shop.adafruit.com/datasheets/WS2812B.pdf" H 2850 4275 50  0001 L TNN
 	1    2750 4650
@@
 F 0 "D3" V 2796 3706 50  0000 R CNN
 F 1 "WS2812B" V 2705 3706 50  0000 R CNN
-F 2 "LED_SMD:LED_WS2812B_PLCC4_5.0x5.0mm_P3.2mm" H 2800 3750 50  0001 L TNN
+F 2 "cnc3018-PCB:myWS2812" H 2800 3750 50  0001 L TNN
 F 3 "https://cdn-shop.adafruit.com/datasheets/WS2812B.pdf" H 2850 3675 50  0001 L TNN
 	1    2750 4050
@@
 F 0 "D2" V 2796 3106 50  0000 R CNN
 F 1 "WS2812B" V 2705 3106 50  0000 R CNN
-F 2 "LED_SMD:LED_WS2812B_PLCC4_5.0x5.0mm_P3.2mm" H 2800 3150 50  0001 L TNN
+F 2 "cnc3018-PCB:myWS2812" H 2800 3150 50  0001 L TNN
 F 3 "https://cdn-shop.adafruit.com/datasheets/WS2812B.pdf" H 2850 3075 50  0001 L TNN
 	1    2750 3450
@@
 $EndComp
 $Comp
-L LED:WS2812B D1
-U 1 1 61F5E592
-P 2750 2850
-F 0 "D1" V 2796 2506 50  0000 R CNN
-F 1 "WS2812B" V 2705 2506 50  0000 R CNN
-F 2 "LED_SMD:LED_WS2812B_PLCC4_5.0x5.0mm_P3.2mm" H 2800 2550 50  0001 L TNN
-F 3 "https://cdn-shop.adafruit.com/datasheets/WS2812B.pdf" H 2850 2475 50  0001 L TNN
-	1    2750 2850
-	0    -1   -1   0
-$EndComp
-$Comp
 L Connector_Generic:Conn_01x03 J1
 U 1 1 61F61BA9
-P 2750 2200
-F 0 "J1" V 2714 2012 50  0000 R CNN
-F 1 "Conn_01x03" V 2800 2000 50  0000 R CNN
-F 2 "cnc3018-PCB:my3pin" H 2750 2200 50  0001 C CNN
-F 3 "~" H 2750 2200 50  0001 C CNN
-	1    2750 2200
+P 2750 1800
+F 0 "J1" V 2714 1612 50  0000 R CNN
+F 1 "Conn_01x03" V 2800 1600 50  0000 R CNN
+F 2 "cnc3018-PCB:my3pin" H 2750 1800 50  0001 C CNN
+F 3 "~" H 2750 1800 50  0001 C CNN
+	1    2750 1800
 	0    -1   -1   0
 $EndComp
@@
 $EndComp
 Wire Wire Line
-	2750 2400 2750 2550
-Wire Wire Line
 	2750 4950 2750 5150
-Wire Wire Line
-	2850 5150 2850 5050
-Wire Wire Line
-	2850 5050 3050 5050
-Wire Wire Line
-	3050 5050 3050 4650
-Wire Wire Line
-	3050 2500 2850 2500
-Wire Wire Line
-	2850 2500 2850 2400
-Connection ~ 3050 2850
-Wire Wire Line
-	3050 2850 3050 2500
 Connection ~ 3050 3450
-Wire Wire Line
-	3050 3450 3050 2850
 Connection ~ 3050 4050
 Wire Wire Line
@@
 	3050 4650 3050 4050
 Wire Wire Line
-	2650 5150 2650 5050
-Wire Wire Line
-	2650 5050 2450 5050
-Wire Wire Line
 	2450 5050 2450 4650
-Wire Wire Line
-	2450 2500 2650 2500
-Wire Wire Line
-	2650 2500 2650 2450
-Connection ~ 2450 2850
-Wire Wire Line
-	2450 2850 2450 2500
 Connection ~ 2450 3450
-Wire Wire Line
-	2450 3450 2450 2850
 Connection ~ 2450 4050
 Wire Wire Line
@@
 L Connector_Generic:Conn_01x01 J4
 U 1 1 61F66634
-P 3500 2500
-F 0 "J4" H 3580 2542 50  0000 L CNN
-F 1 "Conn_01x01" H 3580 2451 50  0000 L CNN
-F 2 "cnc3018-PCB:my1pin" H 3500 2500 50  0001 C CNN
-F 3 "~" H 3500 2500 50  0001 C CNN
-	1    3500 2500
+P 3400 2250
+F 0 "J4" H 3480 2292 50  0000 L CNN
+F 1 "Conn_01x01" H 3480 2201 50  0000 L CNN
+F 2 "cnc3018-PCB:my1pin" H 3400 2250 50  0001 C CNN
+F 3 "~" H 3400 2250 50  0001 C CNN
+	1    3400 2250
 	1    0    0    -1
 $EndComp
@@
 L Connector_Generic:Conn_01x01 J3
 U 1 1 61F68801
-P 3500 2400
-F 0 "J3" H 3580 2442 50  0000 L CNN
-F 1 "Conn_01x01" H 3580 2351 50  0000 L CNN
-F 2 "cnc3018-PCB:my1pin" H 3500 2400 50  0001 C CNN
-F 3 "~" H 3500 2400 50  0001 C CNN
-	1    3500 2400
+P 3400 2150
+F 0 "J3" H 3480 2192 50  0000 L CNN
+F 1 "Conn_01x01" H 3480 2101 50  0000 L CNN
+F 2 "cnc3018-PCB:my1pin" H 3400 2150 50  0001 C CNN
+F 3 "~" H 3400 2150 50  0001 C CNN
+	1    3400 2150
 	1    0    0    -1
 $EndComp
 Wire Wire Line
-	2650 2450 3150 2450
+	3050 3450 3050 2850
+Connection ~ 3050 2850
 Wire Wire Line
-	3150 2450 3150 2400
+	2450 3450 2450 2850
+Connection ~ 2450 2850
+$Comp
+L LED:WS2812B D1
+U 1 1 61F5E592
+P 2750 2850
+F 0 "D1" V 2796 2506 50  0000 R CNN
+F 1 "WS2812B" V 2705 2506 50  0000 R CNN
+F 2 "cnc3018-PCB:myWS2812" H 2800 2550 50  0001 L TNN
+F 3 "https://cdn-shop.adafruit.com/datasheets/WS2812B.pdf" H 2850 2475 50  0001 L TNN
+	1    2750 2850
+	0    -1   -1   0
+$EndComp
 Wire Wire Line
-	3150 2400 3300 2400
-Connection ~ 2650 2450
+	2750 2000 2750 2550
 Wire Wire Line
-	2650 2450 2650 2400
+	3050 5000 2650 5000
 Wire Wire Line
-	3050 2500 3300 2500
-Connection ~ 3050 2500
+	2650 5000 2650 5150
+Wire Wire Line
+	3050 5000 3050 4650
+Wire Wire Line
+	2450 5050 2850 5050
+Wire Wire Line
+	2850 5050 2850 5150
+Wire Wire Line
+	2450 2150 2850 2150
+Wire Wire Line
+	2850 2150 2850 2000
+Wire Wire Line
+	2450 2150 2450 2850
+Wire Wire Line
+	3050 2250 2650 2250
+Wire Wire Line
+	2650 2250 2650 2000
+Wire Wire Line
+	3050 2250 3050 2850
+Wire Wire Line
+	3050 2250 3200 2250
+Connection ~ 3050 2250
+Wire Wire Line
+	2850 2150 3200 2150
+Connection ~ 2850 2150
 $EndSCHEMATC
