File: docs/kiCad/board/bilgeAlarm.kicad_pcb (KiCad board)
At the start: 2 copper layers, 111.8 x 88.9 mm, 67 parts, among them J1 PUMP IN, J10 LCD_SDA, J11 LCD_SCL, J12 LCD_GND, J13 ALARM+, J14 ALARM-, J15 LED_GND, J16 LED_GND, J17 LED_DATA, J18 LED_DATA, J19 LED_5V, J2 PUMP2 IN, J20 LED_5V, J21 AUX, J22 AUX, J23 AUX, J24 AUX, J25 AUX, J26 AUX, J27 AUX, J28 AUX, J29 AUX, J3 PUMP OUT, J30 AUX, J31 AUX, J32 AUX, J33 AUX, J34 AUX, J35 AUX, J36 AUX, J37 AUX, J38 AUX, J39 AUX, J4 12V, J40 AUX, J41 AUX, J5 GND, J6 LED_5V, J7 LED_DATA, J8 LED_GND, J9 LCD_5V, K1 RELAY, M1 BUCK01, M2 SD_TYP0, Q1 IRLZ44N, Q2 BCS547, SW1 POWER, SW2 BUTTON1, SW3 BUTTON2, SW4 BUTTON3, U1 ESP32_DEV_0

Commit message: kicad - commit reworked PCB board using my new symbols and 3d footprints
Parts:
- removed J10: LCD_SDA, cnc3018-PCB:my1pin
- removed J11: LCD_SCL, cnc3018-PCB:my1pin
- removed J12: LCD_GND, cnc3018-PCB:my1pin
- removed J13: ALARM+, cnc3018-PCB:my1pin
- removed J14: ALARM-, cnc3018-PCB:my1pin
- removed J15, J16: LED_GND, cnc3018-PCB:my1pin
- removed J17, J18: LED_DATA, cnc3018-PCB:my1pin
- removed J19, J20: LED_5V, cnc3018-PCB:my1pin
- removed J4: 12V, cnc3018-PCB:my1pin
- removed J5: GND, cnc3018-PCB:my1pin
- added REF**: myLCD_2x16_dimensions, 0_my_footprints:myLCD_2x16_dimensions, F.Cu at (31.8, -52.7)
- added REF**: myMountingHole_3.2mm_M3, 0_my_footprints:myMountingHole_3.2mm_M3, F.Cu at (34.3, -55.2)
- added REF**: myMountingHole_3.2mm_M3, 0_my_footprints:myMountingHole_3.2mm_M3, F.Cu at (109.2, -55.2)
- added REF**: myMountingHole_3.2mm_M3, 0_my_footprints:myMountingHole_3.2mm_M3, F.Cu at (109.2, -86.2)
- added REF**: myMountingHole_3.2mm_M3, 0_my_footprints:myMountingHole_3.2mm_M3, F.Cu at (34.3, -86.2)
- added REF**: myMountingHole_3.2mm_M3, 0_my_footprints:myMountingHole_3.2mm_M3, F.Cu at (3.17, -85.7)
- added REF**: myMountingHole_3.2mm_M3, 0_my_footprints:myMountingHole_3.2mm_M3, F.Cu at (108.6, -3.17)
- added REF**: myMountingHole_3.2mm_M3, 0_my_footprints:myMountingHole_3.2mm_M3, F.Cu at (3.17, -3.17)
- C1: footprint cnc3018-PCB:my2pin -> 0_my_footprints:CP_my100uf
- C2: footprint cnc3018-PCB:my2pin -> 0_my_footprints:CP_my10uf
- D1, D2: footprint cnc3018-PCB:mySkip2 -> 0_my_footprints:myDiodeSchotsky
- J1: value PUMP IN -> BA_POWER; footprint cnc3018-PCB:my1pin -> 0_my_footprints:myTerminalBlock_5.08x02
- J2: value PUMP2 IN -> PUMPS; footprint cnc3018-PCB:my1pin -> 0_my_footprints:myTerminalBlock_5.08x03
- J3: value PUMP OUT -> ALARM; footprint cnc3018-PCB:my1pin -> 0_my_footprints:myTerminalBlock_5.08x02
- J6: value LED_5V -> LEDS; footprint cnc3018-PCB:my1pin -> 0_my_footprints:myPinSocket_1x03
- J7: value LED_DATA -> LEDS OUT; footprint cnc3018-PCB:my1pin -> 0_my_footprints:myPinSocket_1x03
- J8: value LED_GND -> LEDS IN; footprint cnc3018-PCB:my1pin -> 0_my_footprints:myPinSocket_1x03
- J9: value LCD_5V -> LCD; footprint cnc3018-PCB:my1pin -> 0_my_footprints:myPinSocket_1x04
- K1: footprint Relay_THT:Relay_SPDT_SANYOU_SRD_Series_Form_C -> 0_my_footprints:myRelay
- M1: footprint cnc3018-PCB:BUCK01 -> 0_my_footprints:myMini360BuckConverter
- M2: footprint cnc3018-PCB:my6Pin -> 0_my_footprints:SDCardReader
- Q1: footprint Package_TO_SOT_THT:TO-220-3_Vertical -> 0_my_footprints:myTO-220-3
- R1, R10, R11, R13, R2, R3, R4, R5, R6, R7, R8, R9: footprint cnc3018-PCB:myResistor -> 0_my_footprints:myResistor
- SW1: footprint cnc3018-PCB:SW_DPDT_BLUE_LEVER -> 0_my_footprints:mySwitchToggleSPDT
- SW2, SW3, SW4: footprint cnc3018-PCB:BUTTON -> 0_my_footprints:myButton
- U1: footprint cnc3018-PCB:ESP32-DEV_0 -> 0_my_footprints:myESP32DEV0
- moved J7 62.3 mm to (20.3, -85.1), turned to 90 degrees
- moved J8 55.9 mm to (20.3, -78.7), turned to 90 degrees
- moved J3 53.3 mm to (5.08, -71.1), turned to 270 degrees
- moved J1 21.0 mm to (5.08, -33.7), turned to 270 degrees
- moved J6 5.08 mm to (20.3, -22.9), turned to 90 degrees
- moved J9 2.63 mm to (40.0, -81.9)
- moved D1 2.62 mm to (10.2, -64.1)
- moved J2 0.64 mm to (5.08, -23.5), turned to 270 degrees
Connections:
- J1 pad 1: PUMP_IN -> RAW_12V
- J3 pad 1: PUMP_OUT -> Net-(D1-Pad2)
- J6 pad 1: +5V -> GND
- J7 pad 1: LED_DATA -> GND
- J9 pad 1: +5V -> GND
Routing:
- net Net-(J7-Pad2): track 0.00 -> 6.30 mm
- net Net-(J17-Pad1): track 6.30 -> 0.00 mm
- net +12V: track 25.3 -> 31.3 mm, vias 1 -> 0
- net PUMP_IN: track 65.3 -> 70.6 mm, vias 1 -> 0
- net RAW_12V: track 40.9 -> 37.4 mm, vias 1 -> 0
- net +5V: track 174.8 -> 172.1 mm, vias 6 -> 5
- net PUMP_OUT: track 52.4 -> 52.5 mm, vias 2 -> 0
- net GND: vias 6 -> 3
- net +3V3: vias 10 -> 9
- net (no net): vias 7 -> 0
Other:
- board text removed: "January 2022"
- board text removed: "Patrick Horton"
- board text removed: "bilgeAlarm v1.0"
